Commit message: hw2

File: catkin_ws/src/flower_observer/urdf/moving_realsense2.urdf.xacro (robot description, xacro)
@@ -1,10 +1,13 @@
 <?xml version="1.0"?>
 <robot name="realsense2_camera" xmlns:xacro="http://ros.org/wiki/xacro">
-  <xacro:arg name="use_nominal_extrinsics" default="false"/>
   <xacro:include filename="$(find flower_observer)/urdf/_d435.urdf.xacro" />
+  <xacro:include filename="$(find realsense2_description)/urdf/_l515.urdf.xacro" />
   <link name="base_link" />
-  <xacro:sensor_d435 parent="base_link">
+  <xacro:sensor_d435 parent="base_link" name="d435">
     <origin xyz="0 0 0" rpy="0 0 3.1415"/>
   </xacro:sensor_d435>
+  <xacro:sensor_l515 parent="base_link" name="l515">
+    <origin xyz="0 0 0" rpy="0 0 0"/>
+  </xacro:sensor_l515>
 </robot>
 <!-- <xacro:sensor_d435 parent="base_link" use_nominal_extrinsics="$(arg use_nominal_extrinsics)"  add_plug="$(arg add_plug)"> -->

Commit message: add project

File: catkin_ws/src/flower_observer/urdf/moving_realsense2.urdf.xacro (robot description, xacro)
@@ -1,13 +1,16 @@
 <?xml version="1.0"?>
 <robot name="realsense2_camera" xmlns:xacro="http://ros.org/wiki/xacro">
-  <xacro:include filename="$(find flower_observer)/urdf/_d435.urdf.xacro" />
-  <xacro:include filename="$(find realsense2_description)/urdf/_l515.urdf.xacro" />
+  <!-- <xacro:include filename="$(find flower_observer)/urdf/_d435.urdf.xacro" /> -->
+  <!-- <xacro:include filename="$(find realsense2_description)/urdf/_l515.urdf.xacro" /> -->
   <link name="base_link" />
-  <xacro:sensor_d435 parent="base_link" name="d435">
-    <origin xyz="0 0 0" rpy="0 0 3.1415"/>
-  </xacro:sensor_d435>
-  <xacro:sensor_l515 parent="base_link" name="l515">
+  <!-- <xacro:sensor_d435 parent="base_link" name="d435">
     <origin xyz="0 0 0" rpy="0 0 0"/>
-  </xacro:sensor_l515>
+  </xacro:sensor_d435> --> -->
+  <xacro:include filename="$(find realsense_gazebo_description)/urdf/_d435i.urdf.xacro"/>
+  <xacro:sensor_d435i parent="base_link" name="D435i_camera" topics_ns="D435i_camera" enable_pointCloud="true">
+    <origin xyz="0.0 0.0 0.0" rpy="0.0 0.0 0.0"/>
+  </xacro:sensor_d435i>
+  <!-- <xacro:sensor_l515 parent="base_link" name="l515">
+    <origin xyz="0 0 0" rpy="0 0 0"/>
+  </xacro:sensor_l515> -->
 </robot>
-<!-- <xacro:sensor_d435 parent="base_link" use_nominal_extrinsics="$(arg use_nominal_extrinsics)"  add_plug="$(arg add_plug)"> -->
